File: hardware/DaisyPatchSMThingie.kicad_pcb (KiCad board)
At the start: 2 copper layers, 236.2 x 124.5 mm, 64 parts, among them J1 01x02 PIN CONNECTOR, J10 STEREO 3.5mm, J11 MONO 3.5mm, J12 MONO 3.5mm, J13 STEREO 3.5mm, J14 MONO 3.5mm, J15 MONO 3.5mm, J16 STEREO 3.5mm, J17 STEREO 3.5mm, J18 JST 01x03, J19 JST 01x03, J2 EuroRack_Bus_Connector_16_PIN, J20 MONO 3.5mm, J21 MONO 3.5mm, J22 MONO 3.5mm, J23 MONO 3.5mm, J3 Conn_02x20_Odd_Even, J4 02x17 PIN CONNECTOR, J6 Yamaichi PJS008-4100-0-VE, J7 01x06 PIN CONNECTOR, J8 JST 01x03, J9 JST 01x03, SW1 EN11C, SW2 SW_PUSH_6mm, SW3 SW_PUSH_6mm, SW4 SW_PUSH_6mm, SW5 SW_PUSH_6mm, U1 Daisy_Patch_SM, U2 H11L1, U3 SSD1306 0.96" OLED I2C

Commit message: Initial Revision A
Parts:
- removed D4: 1N4148, Diode_THT:D_DO-35_SOD27_P7.62mm_Horizontal
- removed R6: 4k7Ω, Resistor_THT:R_Axial_DIN0204_L3.6mm_D1.6mm_P7.62mm_Horizontal
- removed R7, R8, R9: 47kΩ, Resistor_THT:R_Axial_DIN0204_L3.6mm_D1.6mm_P7.62mm_Horizontal
- added D3: 1N4148, Diode_THT:D_DO-35_SOD27_P7.62mm_Horizontal, F.Cu at (113.0, 88.9)
- added F1: Fuse, Fuses:65600001409, F.Cu at (45.5, 78.7)
- added F2: Fuse, Fuses:65600001409, F.Cu at (45.5, 66.7)
- added J24: STEREO 3.5mm, Desval:Jack_3.5mm_QingPu_WQP-PJ366ST_Vertical, F.Cu at (118.1, 52.1)
- added J25: MONO 3.5mm, Desval:Jack_3.5mm_QingPu_WQP-PJ398SM_Vertical, F.Cu at (130.8, 52.1)
- added J26: MONO 3.5mm, Desval:Jack_3.5mm_QingPu_WQP-PJ398SM_Vertical, F.Cu at (141.0, 52.1)
- added J27: STEREO 3.5mm, Desval:Jack_3.5mm_QingPu_WQP-PJ366ST_Vertical, F.Cu at (73.7, 52.1)
- added J28: MONO 3.5mm, Desval:Jack_3.5mm_QingPu_WQP-PJ398SM_Vertical, F.Cu at (86.4, 52.1)
- added J29: MONO 3.5mm, Desval:Jack_3.5mm_QingPu_WQP-PJ398SM_Vertical, F.Cu at (96.5, 52.1)
- added J30: JST 01x03, Connector_JST:JST_XH_B3B-XH-A_1x03_P2.50mm_Vertical, F.Cu at (60.3, 71.1)
- added J31: JST 01x03, Connector_JST:JST_XH_B3B-XH-A_1x03_P2.50mm_Vertical, F.Cu at (60.3, 80.6)
- added J32: EuroRack_Bus_Connector_10_PIN, Connector_IDC:IDC-Header_2x05_P2.54mm_Vertical, F.Cu at (50.8, 50.8)
- added S1: EG2219, Switches:SW_EG2219, F.Cu at (35.6, 55.9)
- C1: value 10µF -> 100nF; footprint Capacitor_THT:CP_Radial_D5.0mm_P2.00mm -> Capacitor_THT:C_Disc_D4.3mm_W1.9mm_P5.00mm
- C3: value 100nF -> 10µF; footprint Capacitor_THT:C_Disc_D4.3mm_W1.9mm_P5.00mm -> Capacitor_THT:CP_Radial_D5.0mm_P2.00mm
- J1: value 01x02 PIN CONNECTOR -> Conn_02x20_Odd_Even; footprint Connector_PinHeader_2.54mm:PinHeader_1x02_P2.54mm_Vertical -> Connector_PinHeader_2.54mm:PinHeader_2x20_P2.54mm_Vertical
- J10, J13, J16, J17: value STEREO 3.5mm -> MONO 3.5mm; footprint Desval:Jack_3.5mm_QingPu_WQP-PJ366ST_Vertical -> Desval:Jack_3.5mm_QingPu_WQP-PJ398SM_Vertical
- J18, J19: value JST 01x03 -> MONO 3.5mm; footprint Connector_JST:JST_XH_B3B-XH-A_1x03_P2.50mm_Vertical -> Desval:Jack_3.5mm_QingPu_WQP-PJ398SM_Vertical
- J2: value EuroRack_Bus_Connector_16_PIN -> 02x15 PIN CONNECTOR; footprint Connector_IDC:IDC-Header_2x08_P2.54mm_Vertical -> Connector_PinHeader_2.54mm:PinHeader_2x15_P2.54mm_Vertical
- J3: value Conn_02x20_Odd_Even -> 01x02 PIN CONNECTOR; footprint Connector_PinHeader_2.54mm:PinHeader_2x20_P2.54mm_Vertical -> Connector_PinHeader_2.54mm:PinHeader_1x02_P2.54mm_Vertical
- J4: value 02x17 PIN CONNECTOR -> Yamaichi PJS008-4100-0-VE; footprint Connector_PinHeader_2.54mm:PinHeader_2x17_P2.54mm_Vertical -> Desval-Micro_SD_Sockets:Yamaichi PJS00841000VE
- J6: value Yamaichi PJS008-4100-0-VE -> JST 01x03; footprint Desval-Micro_SD_Sockets:Yamaichi PJS00841000VE -> Connector_JST:JST_XH_B3B-XH-A_1x03_P2.50mm_Vertical
- J7: value 01x06 PIN CONNECTOR -> JST 01x03; footprint Connector_PinHeader_2.54mm:PinHeader_1x06_P2.54mm_Vertical -> Connector_JST:JST_XH_B3B-XH-A_1x03_P2.50mm_Vertical
- J8, J9: value JST 01x03 -> STEREO 3.5mm; footprint Connector_JST:JST_XH_B3B-XH-A_1x03_P2.50mm_Vertical -> Desval:Jack_3.5mm_QingPu_WQP-PJ366ST_Vertical
- R1, R2: value 1kΩ -> 4k7Ω
- R10: value 47kΩ -> 220Ω
- R11: value 47kΩ -> 270Ω
- R3: value 220Ω -> 1kΩ
- R4: value 4k7Ω -> 1kΩ
- R5: value 270Ω -> 1kΩ
- U2: value H11L1 -> SSD1306 0.96" OLED I2C; footprint Package_DIP:DIP-6_W7.62mm_Socket_LongPads -> Desval:0.96 Inch OLED I2C Display Module
- U3: value SSD1306 0.96" OLED I2C -> H11L1; footprint Desval:0.96 Inch OLED I2C Display Module -> Package_DIP:DIP-6_W7.62mm_Socket_LongPads
- moved J2 207.5 mm to (233.7, 109.2)
- moved J1 190.8 mm to (35.6, 109.2)
- moved C3 112.5 mm to (64.8, 62.9), turned to 90 degrees
- moved J4 96.6 mm to (31.0, 95.9), turned to 180 degrees
- moved U3 96.5 mm to (111.8, 68.6)
- moved J13 88.9 mm to (163.8, 69.8)
- moved JP1 81.8 mm to (96.5, 85.7)
- moved JP2 81.8 mm to (96.5, 76.8)
- moved JP3 81.8 mm to (96.5, 80.0)
- moved JP4 81.8 mm to (96.5, 88.9)
- moved J11 81.4 mm to (167.6, 87.6)
- moved J10 80.1 mm to (154.9, 87.6)
- moved R5 78.2 mm to (106.7, 81.3), turned to -90 degrees
- moved R11 77.1 mm to (124.5, 81.3)
- moved C1 74.9 mm to (127.0, 68.7), turned to -90 degrees
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Connections:
- C1 pad 1: +12V -> +3V3
- C2 pad 1: GND -> +12V
- C2 pad 2: -12V -> GND
- C3 pad 1: +3.3V -> GND
- C3 pad 2: GND -> -12V
- J1 pad 1: Net-(J1-Pin_1) -> -12V
- J1 pad 2: Net-(J1-Pin_2) -> SDMMC_CLK
- J10 pad T: AUDIO_IN_L -> GATE_OUT_1
- J11 pad T: AUDIO_IN_L -> GATE_OUT_2
- J12 pad T: AUDIO_IN_R -> GATE_IN_1
- J12 pad TN: AUDIO_IN_L -> unconnected-(J12-SW-PadTN)
- J13 pad T: AUDIO_OUT_L -> GATE_IN_2
- J14 pad T: AUDIO_OUT_L -> CV_OUT_1
- J15 pad T: AUDIO_OUT_R -> CV_OUT_2
- J16 pad T: MIDI_IN_TIP -> CV_1
- J17 pad T: MIDI_OUT_5 -> CV_2
- J2 pad 1: -12V -> RV_A
- J2 pad 10: +12V -> ENCODER_A
- J2 pad 11: unconnected-(J2-+5V-Pad11) -> ENCODER_B
- J2 pad 12: unconnected-(J2-+5V-Pad12) -> ENCODER_B
- J2 pad 13: unconnected-(J2-CV-Pad13) -> ENCODER_SW
- J2 pad 14: unconnected-(J2-CV-Pad14) -> ENCODER_SW
- J2 pad 15: unconnected-(J2-GATE-Pad15) -> SW_A
- J2 pad 16: unconnected-(J2-GATE-Pad16) -> SW_A
- J2 pad 2: -12V -> RV_A
- J2 pad 3: GND -> RV_B
- J2 pad 4: GND -> RV_B
- J2 pad 5: GND -> RV_C
- J2 pad 6: GND -> RV_C
- J2 pad 7: GND -> RV_D
- J2 pad 8: GND -> RV_D
- J2 pad 9: +12V -> ENCODER_A
- J20 pad T: JA_T -> CV_5
- J20 pad TN: JA_TN -> unconnected-(J20-SW-PadTN)
- J21 pad T: JB_T -> CV_6
- J21 pad TN: JB_TN -> unconnected-(J21-SW-PadTN)
- J22 pad T: JC_T -> CV_7
- J22 pad TN: JC_TN -> unconnected-(J22-SW-PadTN)
- J23 pad T: JD_T -> CV_8
- J23 pad TN: JD_TN -> unconnected-(J23-SW-PadTN)
- J3 pad 1: -12V -> Net-(J3-Pin_1)
- J3 pad 2: SDMMC_CLK -> Net-(J3-Pin_2)
- J4 pad 1: RV_A -> SDMMC_D2
- J4 pad 10: ENCODER_A -> GND
- J4 pad 11: ENCODER_B -> GND
- J4 pad 12: ENCODER_B -> GND
- J4 pad 2: RV_A -> SDMMC_D3
- J4 pad 3: RV_B -> SDMMC_CMD
- J4 pad 4: RV_B -> +3V3
- J4 pad 5: RV_C -> SDMMC_CLK
- J4 pad 6: RV_C -> GND
- J4 pad 7: RV_D -> SDMMD_D0
- J4 pad 8: RV_D -> SDMMC_D1
- J4 pad 9: ENCODER_A -> GND
- J6 pad 1: MSD_DAT2 -> MIDI_IN_4
- J6 pad 2: MSD_DAT3 -> GND
- J6 pad 3: MSD_CMD -> MIDI_IN_5
- J7 pad 1: MSD_CLK -> MIDI_OUT_4
- J7 pad 2: MSD_CMD -> GND
- J7 pad 3: MSD_DAT0 -> MIDI_OUT_5
- R1 pad 1: Net-(J1-Pin_1) -> +3V3
- R1 pad 2: Net-(D1-A) -> SCL
- R10 pad 1: +3.3V -> MIDI_IN_4
- R10 pad 2: MSD_DAT0 -> Net-(D3-K)
- R11 pad 1: +3.3V -> +3V3
- R11 pad 2: MSD_CMD -> MIDI_RX
- R13 pad 1: +3.3V -> +3V3
- R2 pad 1: Net-(J1-Pin_2) -> +3V3
- R2 pad 2: Net-(D2-A) -> SDA
- R3 pad 1: MIDI_IN_4 -> Net-(J3-Pin_1)
- R3 pad 2: Net-(D4-K) -> Net-(D1-A)
- R4 pad 1: unconnected-(R4-Pad1) -> Net-(J3-Pin_2)
- R4 pad 2: SCL -> Net-(D2-A)
- R5 pad 1: +3.3V -> AUDIO_OUT_L
- R5 pad 2: MIDI_RX -> AUDIO_OUT_R
- RV1 pad 3: +3.3VA -> +3V3
- RV2 pad 3: +3.3VA -> +3V3
- RV3 pad 3: +3.3VA -> +3V3
- RV4 pad 3: +3.3VA -> +3V3
- U1 pad A2: unconnected-(U1-UART_RX-PadA2) -> UART_RX
- U1 pad A3: unconnected-(U1-UART_TX-PadA3) -> UART_TX
- U1 pad A8: unconnected-(U1-USB_DM-PadA8) -> USB_DM
- U1 pad A9: unconnected-(U1-USB_DP-PadA9) -> USB_DP
- U1 pad B1: unconnected-(U1-AUDIO_OUT_R-PadB1) -> AUDIO_OUT_R
- U1 pad B10: unconnected-(U1-GATE_IN_1-PadB10) -> GATE_IN_1
- U1 pad B2: unconnected-(U1-AUDIO_OUT_L-PadB2) -> AUDIO_OUT_L
- U1 pad B3: unconnected-(U1-AUDIO_IN_R-PadB3) -> AUDIO_IN_R
- U1 pad B4: unconnected-(U1-AUDIO_IN_L-PadB4) -> AUDIO_IN_L
- U1 pad B5: unconnected-(U1-GATE_OUT_1-PadB5) -> GATE_OUT_1
- U1 pad B6: unconnected-(U1-GATE_OUT_2-PadB6) -> GATE_OUT_2
- U1 pad B7: unconnected-(U1-I2C1_SCL-PadB7) -> SCL
- U1 pad B8: unconnected-(U1-I2C1_SDA-PadB8) -> SDA
- U1 pad B9: unconnected-(U1-GATE_IN_2-PadB9) -> GATE_IN_2
- U1 pad C1: unconnected-(U1-CV_OUT_2-PadC1) -> CV_OUT_2
- U1 pad C10: unconnected-(U1-CV_OUT_1-PadC10) -> CV_OUT_1
- U1 pad C2: unconnected-(U1-CV4-PadC2) -> CV_4
- U1 pad C3: unconnected-(U1-CV3-PadC3) -> CV_3
- U1 pad C4: unconnected-(U1-CV2-PadC4) -> CV_2
- U1 pad C5: unconnected-(U1-CV1-PadC5) -> CV_1
- U1 pad C6: unconnected-(U1-CV5-PadC6) -> CV_5
- U1 pad C7: unconnected-(U1-CV6-PadC7) -> CV_6
- U1 pad C8: unconnected-(U1-CV7-PadC8) -> CV_7
- U1 pad C9: unconnected-(U1-CV8-PadC9) -> CV_8
- U1 pad D1: unconnected-(U1-SPI_NSS-PadD1) -> SPI_CS
- U1 pad D10: unconnected-(U1-SPI_SCK-PadD10) -> SPI_SCK
- U1 pad D2: unconnected-(U1-SDMMC_D3-PadD2) -> SDMMC_D3
- U1 pad D3: unconnected-(U1-SDMMC_D2-PadD3) -> SDMMC_D2
- U1 pad D4: unconnected-(U1-SDMMC_D1-PadD4) -> SDMMC_D1
- U1 pad D5: unconnected-(U1-SDMMC_D0-PadD5) -> SDMMD_D0
- U1 pad D6: unconnected-(U1-SDMMC_CK-PadD6) -> SDMMC_CLK
- U1 pad D7: unconnected-(U1-SDMMC_CMD-PadD7) -> SDMMC_CMD
- U1 pad D8: unconnected-(U1-SPI_MISO-PadD8) -> SPI_MISO
- U1 pad D9: unconnected-(U1-SPI_MOSI-PadD9) -> SPI_MOSI
- U2 pad 1: Net-(D4-K) -> GND
- U2 pad 2: MIDI_IN_5 -> +3V3
- U2 pad 3: unconnected-(U2-Pad3) -> SCL
- U2 pad 4: MIDI_RX -> SDA
- U3 pad 1: GND -> Net-(D3-K)
- U3 pad 2: +3.3V -> MIDI_IN_5
- U3 pad 3: SCL -> unconnected-(U3-Pad3)
- U3 pad 4: SDA -> MIDI_RX
Routing:
- net GND: track 0.00 -> 1123.9 mm
- net SCL: track 0.00 -> 405.5 mm, vias 0 -> 4
- net SDA: track 0.00 -> 384.4 mm, vias 0 -> 5
- net +3V3: track 0.00 -> 374.8 mm, vias 0 -> 4
- net CV_8: track 0.00 -> 261.9 mm, vias 0 -> 2
- net CV_7: track 0.00 -> 246.5 mm, vias 0 -> 6
- net CV_4: track 0.00 -> 236.6 mm, vias 0 -> 1
- net CV_3: track 0.00 -> 219.1 mm, vias 0 -> 1
- net CV_5: track 0.00 -> 217.3 mm, vias 0 -> 1
- net AUDIO_IN_R: track 0.00 -> 216.0 mm, vias 0 -> 2
- net CV_6: track 0.00 -> 215.8 mm, vias 0 -> 2
- net CV_1: track 0.00 -> 215.2 mm, vias 0 -> 2
- net AUDIO_OUT_L: track 0.00 -> 215.0 mm, vias 0 -> 2
- net CV_2: track 0.00 -> 215.0 mm, vias 0 -> 3
- net CV_OUT_2: track 0.00 -> 213.5 mm, vias 0 -> 1
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Other:
- board text added: "+12V"
- board text added: "-12V"
- board text added: "3V3"
- board text added: "5V"
- board text added: "BTN A"
- board text added: "BTN B"
- board text added: "BTN C"
- board text added: "BTN D"
- board text added: "BTN E"
- board text added: "CS"
- board text added: "CV 1"
- board text added: "CV 2"
- board text added: "CV 3"
- board text added: "CV 4"
- board text added: "CV 5"
- board text added: "CV 6"
- board text added: "CV 7"
- board text added: "CV 8"
- board text added: "CV OUT 1"
- board text added: "CV OUT 2"
- board text added: "ENC A"
- board text added: "ENC B"
- board text added: "GATE IN 1"
- board text added: "GATE IN 2"
- board text added: "GATE OUT 1"
- board text added: "GATE OUT 2"
- board text added: "GND"
- board text added: "IN L"
- board text added: "IN R"
- board text added: "MIDI RX"
- board text added: "MIDI TX"
- board text added: "MISO"
- board text added: "MOSI"
- board text added: "OUT L"
- board text added: "OUT R"
- board text added: "POT A"
- board text added: "POT B"
- board text added: "POT C"
- board text added: "POT D"
- board text added: "SCK"
- board text added: "SCL"
- board text added: "SDA"
- board text added: "SDCLK"
- board text added: "SDCMD"
- board text added: "SDD 0"
- board text added: "SDD 1"
- board text added: "SDD 2"
- board text added: "SDD 3"
- board text added: "UART RX"
- board text added: "UART TX"
- board text added: "USB DM"
- board text added: "USB DP"
- board text removed: "+5-17VDC"
- board text removed: "3V3A"
- board text removed: "3V3D"
- board text removed: "A0/D15"
- board text removed: "A1/D16"
- board text removed: "A10/D25"
- board text removed: "A11/D28"
- board text removed: "A2/D17"
- board text removed: "A3/D18"
- board text removed: "A4/D19"
- board text removed: "A5/D20"
- board text removed: "A6/D21"
- board text removed: "A7/D22"
- board text removed: "A8/D23"
- board text removed: "A9/D24"
- board text removed: "AGND"
- board text removed: "BUTTONS"
- board text removed: "C"
- board text removed: "CLK"
- board text removed: "CMD"
- board text removed: "CS/D7"
- board text removed: "D"
- board text removed: "D26"
- board text removed: "D27"
- board text removed: "D29"
- board text removed: "D30"
- board text removed: "DAT0"
- board text removed: "DAT1"
- board text removed: "DAT2"
- board text removed: "DAT3"
- board text removed: "DGND"
- board text removed: "E"
- board text removed: "EN"
- board text removed: "IN1"
- board text removed: "IN2"
- board text removed: "JACKS"
- board text removed: "L"
- board text removed: "M"
- board text removed: "MOSI/D10"
- board text removed: "MSIO/D9"
- board text removed: "NC"
- board text removed: "OUT1"
- board text removed: "OUT2"
- board text removed: "POTS"
- board text removed: "R"
- board text removed: "RX/D14"
- board text removed: "S"
- board text removed: "SCK/D8"
- board text removed: "SCL/D11"
- board text removed: "SDA/D12"
- board text removed: "SDCLK/D6"
- board text removed: "SDCMD/D5"
- board text removed: "SDD0/D4"
- board text removed: "SDD1/D3"
- board text removed: "SDD2/D2"
- board text removed: "SDD3/D1"
- board text removed: "T"
- board text removed: "TIP"
- board text removed: "TX/D13"
- board text removed: "USBID/D0"
- board text removed: "VIN"
- board text removed: "X"
