File: hardware/DaisyPatchSMThingie.kicad_sch (KiCad schematic)
At the start: 25 parts, among them J1 01x02 PIN CONNECTOR, J2 EuroRack_Bus_Connector_16_PIN, J3 Conn_02x20_Odd_Even, J4 02x17 PIN CONNECTOR, SW1 EN11C, SW2 SW_PUSH_6mm, SW3 SW_PUSH_6mm, SW4 SW_PUSH_6mm, SW5 SW_PUSH_6mm, U1 Daisy_Patch_SM, U3 SSD1306 0.96" OLED I2C

Commit message: Initial Revision A
Parts:
- removed C1, C2: 10µF, Capacitor_THT:CP_Radial_D5.0mm_P2.00mm, symbol Device:C_Polarized
- removed C4, C5: 100nF, Capacitor_THT:C_Disc_D4.3mm_W1.9mm_P5.00mm, symbol Device:C
- removed J2: EuroRack_Bus_Connector_16_PIN, Connector_IDC:IDC-Header_2x08_P2.54mm_Vertical, symbol EuroRack:EuroRack_Bus_Connector_16_PIN
- added J4: Yamaichi PJS008-4100-0-VE, Desval-Micro_SD_Sockets:Yamaichi PJS00841000VE, symbol Desval-Micro_SD_Sockets:Yamaichi PJS008-4100-0-VE
- J2: renamed from J4; value 02x17 PIN CONNECTOR -> 02x15 PIN CONNECTOR; footprint Connector_PinHeader_2.54mm:PinHeader_2x17_P2.54mm_Vertical -> Connector_PinHeader_2.54mm:PinHeader_2x15_P2.54mm_Vertical; symbol Connector_Generic:Conn_02x17_Odd_Even -> Connector_Generic:Conn_02x15_Odd_Even
- renumbered J3 to J1, J1 to J3, R4 to R1, R6 to R2, R1 to R3, R2 to R4, U3 to U2
Connections:
- net +3.3V is gone; now on net +3V3: U2.2 (VCC)
- net +3.3VA is gone; now on net +5V: RV1.3, RV2.3, RV3.3, RV4.3
- net JA_T is gone; now on net SDA: J2.27 (Pin_27)
- net JA_TN is gone; now on net SDA: J2.28 (Pin_28)
- net JB_T is gone; now on net SCL: J2.29 (Pin_29)
- net JB_TN is gone; now on net SCL: J2.30 (Pin_30)
- net +3V3: now also R1.1, R2.1, J4.4 (VDD)
- net AUDIO_IN_L: now also U1.B4 (AUDIO_IN_L)
- net AUDIO_IN_R: now also U1.B3 (AUDIO_IN_R)
- net AUDIO_OUT_L: now also U1.B2 (AUDIO_OUT_L)
- net AUDIO_OUT_R: now also U1.B1 (AUDIO_OUT_R)
- net CV_1: now also U1.C5 (CV1)
- net CV_2: now also U1.C4 (CV2)
- net CV_3: now also U1.C3 (CV3)
- net CV_4: now also U1.C2 (CV4)
- net CV_5: now also U1.C6 (CV5)
- net CV_6: now also U1.C7 (CV6)
- net CV_7: now also U1.C8 (CV7)
- net CV_8: now also U1.C9 (CV8)
- net CV_OUT_1: now also U1.C10 (CV_OUT_1)
- net CV_OUT_2: now also U1.C1 (CV_OUT_2)
- net GATE_IN_1: now also U1.B10 (GATE_IN_1)
- net GATE_IN_2: now also U1.B9 (GATE_IN_2)
- net GATE_OUT_1: now also U1.B5 (GATE_OUT_1)
- net GATE_OUT_2: now also U1.B6 (GATE_OUT_2)
- net GND: now also J4.10 (MP_2), J4.11 (MP_3), J4.12 (MP_4), J4.6 (VSS), J4.9 (MP_1)
- net MIDI_RX: now also J2.24 (Pin_24)
- net MIDI_TX: now also J2.25 (Pin_25), J2.26 (Pin_26); no longer J2.24 (Pin_24)
- net SCL: now also U1.B7 (I2C1_SCL); no longer J2.25 (Pin_25)
- net SDA: now also U1.B8 (I2C1_SDA); no longer J2.26 (Pin_26)
- net SDMMC_CLK: now also U1.D6 (SDMMC_CK), J4.5 (CLK)
- net SDMMC_CMD: now also U1.D7 (SDMMC_CMD), J4.3 (CMD)
- net SDMMC_D1: now also U1.D4 (SDMMC_D1), J4.8 (DAT1)
- net SDMMC_D2: now also U1.D3 (SDMMC_D2), J4.1 (DAT2)
- net SDMMC_D3: now also U1.D2 (SDMMC_D3), J4.2 (CD/DAT3)
- net SDMMD_D0: now also U1.D5 (SDMMC_D0), J4.7 (DAT0)
- net SPI_CS: now also U1.D1 (SPI_NSS)
- net SPI_MISO: now also J1.18 (Pin_18), U1.D8 (SPI_MISO); no longer J1.20 (Pin_20)
- net SPI_MOSI: now also J1.16 (Pin_16), U1.D9 (SPI_MOSI); no longer J1.18 (Pin_18)
- net SPI_SCK: now also J1.20 (Pin_20), U1.D10 (SPI_SCK); no longer J1.16 (Pin_16)
- net UART_RX: now also U1.A2 (UART_RX)
- net UART_TX: now also U1.A3 (UART_TX)
- net USB_DM: now also U1.A8 (USB_DM)
- net USB_DP: now also U1.A9 (USB_DP)
- removed net JC_T: J2.31 (Pin_31)
- removed net JC_TN: J2.32 (Pin_32)
- removed net JD_T: J2.33 (Pin_33)
- removed net JD_TN: J2.34 (Pin_34)
- no-connect marks 6 -> 0
Other:
- removed sheet SDCard
- added sheet Power (power.kicad_sch)
- moved on the sheet: D1, D2, J1, J3, R1, R2, R3, R4, SW2, SW3, SW4, SW5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
