File: hardware/jacks.kicad_sch (KiCad schematic)
At the start: 12 parts, among them J10 STEREO 3.5mm, J11 MONO 3.5mm, J12 MONO 3.5mm, J13 STEREO 3.5mm, J14 MONO 3.5mm, J15 MONO 3.5mm, J20 MONO 3.5mm, J21 MONO 3.5mm, J22 MONO 3.5mm, J23 MONO 3.5mm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

Commit message: Initial Revision A
Parts:
- added J11, J12, J13, J14, J15, J16, J17, J18, J19, J20: MONO 3.5mm, Desval:Jack_3.5mm_QingPu_WQP-PJ398SM_Vertical, symbol Desval:3.5mm_Mono_Switched_Jack
- added R5: 1kΩ, Resistor_THT:R_Axial_DIN0204_L3.6mm_D1.6mm_P7.62mm_Horizontal, symbol Device:R
- J10: renamed from J20; Label A -> GATEOUT1
- J21: Label B -> CVIN6
- J22: Label C -> CVIN7
- J23: Label D -> CVIN8
- J25: renamed from J11; Label IN L -> IN L(M)
- J28: renamed from J14; Label OUT L -> OUT L(M)
- renumbered J10 to J24, J12 to J26, J13 to J27, J15 to J29, J8 to J30, J9 to J31
Connections:
- net AUDIO_OUT_L: now also J29.TN (SW), R5.1
- net AUDIO_OUT_R: now also R5.2
- net GND: now also J11.S (SHEILD), J12.S (SHEILD), J13.S (SHEILD), J14.S (SHEILD), J15.S (SHEILD), J16.S (SHEILD), J17.S (SHEILD), J18.S (SHEILD), J19.S (SHEILD), J20.S (SHEILD)
- net JA_T renamed GATE_OUT_1
- net JA_TN: no longer names the net of J10.TN (SW)
- net JB_T renamed CV_6
- net JB_TN: no longer names the net of J21.TN (SW)
- net JC_T renamed CV_7
- net JC_TN: no longer names the net of J22.TN (SW)
- net JD_T renamed CV_8
- net JD_TN: no longer names the net of J23.TN (SW)
- new net CV_1: J16.T (SIG)
- new net CV_2: J17.T (SIG)
- new net CV_3: J18.T (SIG)
- new net CV_4: J19.T (SIG)
- new net CV_5: J20.T (SIG)
- new net CV_OUT_1: J14.T (SIG)
- new net CV_OUT_2: J15.T (SIG)
- new net GATE_IN_1: J12.T (SIG)
- new net GATE_IN_2: J13.T (SIG)
- new net GATE_OUT_2: J11.T (SIG)
- no-connect marks 3 -> 16
Other:
- moved on the sheet: J10, J28, J29, J30, J31
