File: hardware/midi.kicad_sch (KiCad schematic)
At the start: 15 parts, among them J16 STEREO 3.5mm, J17 STEREO 3.5mm, J18 JST 01x03, J19 JST 01x03, U2 H11L1

Commit message: Initial Revision A
Parts:
- renumbered C3 to C1, D4 to D3, J18 to J6, J19 to J7, J16 to J8, J17 to J9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
Connections:
- net +3.3V renamed +3V3
