File: hardware/sdcard.kicad_sch (KiCad schematic)
At the start: 7 parts, among them J6 Yamaichi PJS008-4100-0-VE, J7 01x06 PIN CONNECTOR

Commit message: Initial Revision A
Parts:
- removed J6: Yamaichi PJS008-4100-0-VE, Desval-Micro_SD_Sockets:Yamaichi PJS00841000VE, symbol Desval-Micro_SD_Sockets:Yamaichi PJS008-4100-0-VE
- removed J7: 01x06 PIN CONNECTOR, Connector_PinHeader_2.54mm:PinHeader_1x06_P2.54mm_Vertical, symbol Connector_Generic:Conn_01x06
- removed R10, R11, R7, R8, R9: 47kΩ, Resistor_THT:R_Axial_DIN0204_L3.6mm_D1.6mm_P7.62mm_Horizontal, symbol Device:R
